File: Schematics/SMuFF-Backbone/SMuFF-Backbone.kicad_pcb (KiCad board)
At the start: 2 copper layers, 99.6 x 54.1 mm, 61 parts, among them J1 I2C-IN, J10 SW-I2C, J11 Serial-3, J2 I2C-OUT1, J3 Stepper, J4 Printer, J5 SMuFF, J6 Serial2/3, J7 UART, J8 NPX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

Commit message: Updated to 3.30; See README.md
Parts:
- removed A1: Pololu A4988 Socket, Module:Pololu_Breakout-16_15.2x20.3mm
- removed J10: SW-I2C, Connector_JST:JST_XH_B5B-XH-A_1x05_P2.50mm_Vertical
- removed J11: Serial-3, Connector_PinHeader_2.54mm:PinHeader_1x05_P2.54mm_Vertical
- removed R5, R6, R7: 10K, Resistor_SMD:R_0805_2012Metric
- T1: footprint TerminalBlock:TerminalBlock_bornier-2_P5.08mm -> TerminalBlock_Phoenix:TerminalBlock_Phoenix_MKDS-1,5-2-5.08_1x02_P5.08mm_Horizontal
- moved R8 15.0 mm to (146.6, 134.4), turned to 0 degrees
- moved R11 11.0 mm to (128.0, 116.1), turned to 180 degrees
- moved R10 7.37 mm to (146.6, 122.7)
- moved G*** 6.45 mm to (133.6, 130.3)
- moved T1 4.98 mm to (102.7, 88.5), turned to -90 degrees
- moved R1 1.85 mm to (114.7, 125.3), turned to -90 degrees
- moved R2 1.37 mm to (139.0, 111.6)
- moved C2 0.76 mm to (134.9, 111.3)
- moved D2 0.38 mm to (138.8, 109.3)
Connections:
- U2 pad 20: FLASH -> unconnected-(U2-LED13-Pad20)
- U2 pad 21: RESET -> unconnected-(U2-LED14-Pad21)
- U4 pad 1: RESET -> unconnected-(U4-~{RST}-Pad1)
- U4 pad 11: Net-(R6-Pad1) -> unconnected-(U4-D4-Pad11)
- U4 pad 12: FLASH -> unconnected-(U4-D3-Pad12)
- U4 pad 13: SDA -> unconnected-(U4-SDA/D2-Pad13)
- U4 pad 14: SCL -> unconnected-(U4-SCL/D1-Pad14)
Routing:
- net SDA: track 78.1 -> 37.8 mm
- net FLASH: track 39.2 -> 0.00 mm, vias 1 -> 0
- net SCL: track 75.6 -> 36.8 mm
- net +3V3: track 106.8 -> 69.9 mm, vias 2 -> 0
- net Net-(A1-Pad1): track 19.1 -> 0.00 mm
- net Net-(A1-Pad16): track 16.0 -> 0.00 mm
- net RESET: track 14.8 -> 0.00 mm, vias 1 -> 0
- net Net-(A1-Pad15): track 13.6 -> 0.00 mm
- net Net-(A1-Pad9): track 11.8 -> 0.00 mm
- net Net-(A1-Pad2): track 10.4 -> 0.00 mm
- net Net-(A1-Pad7): track 9.75 -> 0.00 mm
- net Net-(U3-I1): track 22.9 -> 14.7 mm
- net Net-(J8-Pin_2): track 16.7 -> 9.98 mm
- net Net-(U4-SCK/D5): track 12.8 -> 19.0 mm
- net Net-(T1-Pin_1): track 17.3 -> 23.1 mm
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Other:
- board size 99.6 x 54.1 mm -> 78.7 x 54.1 mm
- board text added: "3V3 Out"
- board text added: "I2C Addresses PCA9685 @ 0x40"
- board text added: "MP1584EN"
- board text added: "NeoPixels"
- board text added: "RLY"
- board text added: "SMuFF-Backbone © by Technik Gegg 2022-2025"
- board text removed: "3.3V"
- board text removed: "DIR"
- board text removed: "E3-DIP Adapter for SW-I2C/Ser.3"
- board text removed: "EN"
- board text removed: "I2C Addresses PCA9685 @ 0x40 D1 Mini @ 0x41"
- board text removed: "I2C-OUT2 VCC"
- board text removed: "MP1594EN"
- board text removed: "N.C."
- board text removed: "NeoPX"
- board text removed: "Relay"
- board text removed: "SERIAL3"
- board text removed: "SMuFF-Backbone © by Technik Gegg 2022"
- board text removed: "SW I2C"
- board text removed: "V3.3 Out"
