File: Schematics/SMuFF-Backbone/SMuFF-Backbone.kicad_sch (KiCad schematic)
At the start: 58 parts, among them J1 I2C-IN, J10 SW-I2C, J11 Serial-3, J2 I2C-OUT1, J3 Stepper, J4 Printer, J5 SMuFF, J6 Serial2/3, J7 UART, J8 NPX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

Commit message: Updated to 3.30; See README.md
Parts:
- removed A1: Pololu A4988 Socket, Capacitor_SMD:C_1206_3216Metric, symbol Driver_Motor:Pololu_Breakout_A4988
- removed J10: SW-I2C, Connector_JST:JST_XH_B5B-XH-A_1x05_P2.50mm_Vertical, symbol Connector_Generic:Conn_01x05
- removed J11: Serial-3, Connector_PinHeader_2.54mm:PinHeader_1x05_P2.54mm_Vertical, symbol Connector_Generic:Conn_01x05
- removed R5, R6, R7: 10K, Resistor_SMD:R_0805_2012Metric, symbol Device:R
- D1: value (none) -> PWR LED*; footprint (none) -> LED_SMD:LED_1206_3216Metric
- D2: value (none) -> Relay LED*; footprint (none) -> LED_SMD:LED_1206_3216Metric
- J1, J2, J3, J4, J5, J9: symbol Connector:Conn_01x04_Male -> Connector:Conn_01x04_Pin
- J6, J7, J8: symbol Connector:Conn_01x03_Male -> Connector:Conn_01x03_Pin
- RN1, RN2: footprint Resistor_SMD:R_Array_Concave_4x0603 -> Resistor_SMD:R_Array_Convex_4x0603
Connections:
- net SCL: no longer U4.14 (SCL/D1)
- net SDA: no longer U4.13 (SDA/D2)
- net FLASH: no longer names the net of U4.12 (D3)
- net FLASH: no longer U2.20 (LED13)
- net RESET: no longer names the net of U4.1 (~{RST})
- net RESET: no longer U2.21 (LED14)
- no-connect marks 23 -> 21
Other:
- note added: "Jumper 1-2, from PCA9685 Wire 2-3, from Controller"
- note removed: "3.3V"
- note removed: "5V"
- note removed: "E3-DIP SW-I2C Adapter"
- note removed: "Jumper 1-2, from PCA9586 Wire 2-3, from Controller"
- note removed: "for ZAM-Stepper Driver Socket"
