File: Schematics/SMuFF-Connector/SMuFF-Connector/SMuFF-Connector.kicad_pcb (KiCad board)
At the start: 2 copper layers, 89.2 x 32 mm, 20 parts, among them J1 Selector Stepper, J10 Feeder Sensor, J11 NeoPixels, J12 I2C, J13 (Lid Servo), J14 (Cutter Servo), J15 SPARE, J2 Feeder Stepper, J3 Power, J4 Signals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

Commit message: Updated to 3.30; See README.md
Routing:
- net GND: track 18.0 -> 22.2 mm, vias 2 -> 3
- net +5V: track 136.7 -> 132.6 mm
Other:
- outline, holes or cut-outs redrawn
