File: Schematics/SMuFF-Connector/SMuFF-Connector/SMuFF-Connector.kicad_sch (KiCad schematic)
At the start: 18 parts

Commit message: Updated to 3.30; See README.md
Parts:
- H1, H2, H3: value (none) -> MountingHole; footprint (none) -> MountingHole:MountingHole_3mm
- J1: value (none) -> Selector Stepper; footprint (none) -> Connector_JST:JST_PH_B6B-PH-K_1x06_P2.00mm_Vertical
- J10: value (none) -> Feeder Sensor; footprint (none) -> Connector_JST:JST_XH_B3B-XH-A_1x03_P2.50mm_Vertical
- J11: value (none) -> NeoPixels; footprint (none) -> Connector_JST:JST_XH_B3B-XH-A_1x03_P2.50mm_Vertical
- J12: value (none) -> I2C; footprint (none) -> Connector_JST:JST_XH_B4B-XH-A_1x04_P2.50mm_Vertical
- J13: value (none) -> (Lid Servo); footprint (none) -> Connector_PinHeader_2.54mm:PinHeader_1x03_P2.54mm_Vertical
- J14: value (none) -> (Cutter Servo)
- J15: value (none) -> SPARE; footprint (none) -> Connector_JST:JST_XH_B2B-XH-A_1x02_P2.50mm_Vertical
- J2: value (none) -> Feeder Stepper; footprint (none) -> Connector_JST:JST_PH_B6B-PH-K_1x06_P2.00mm_Vertical
- J3: value (none) -> Power; footprint (none) -> Connector_JST:JST_XH_B4B-XH-A_1x04_P2.50mm_Vertical
- J4: value (none) -> Signals; footprint (none) -> Connector_JST:JST_XH_B5B-XH-A_1x05_P2.50mm_Vertical
- J5: value (none) -> Connector 1x20; footprint (none) -> Connector_PinHeader_1.27mm:PinHeader_1x20_P1.27mm_Vertical
- J6: value (none) -> Conn_01x16; footprint (none) -> Connector_PinHeader_1.27mm:PinHeader_1x20_P1.27mm_Vertical
- J7: value (none) -> Selector Motor; footprint (none) -> Connector_JST:JST_XH_B4B-XH-A_1x04_P2.50mm_Vertical
- J8: value (none) -> Feeder Motor; footprint (none) -> Connector_JST:JST_XH_B4B-XH-A_1x04_P2.50mm_Vertical
- J9: value (none) -> Selector Endstop; footprint (none) -> Connector_JST:JST_XH_B3B-XH-A_1x03_P2.50mm_Vertical
