File: Schematics/SMuFF-Relay-Board/Relay-Board.kicad_sch (KiCad schematic)
At the start: 13 parts, among them J1 JST XH, J2 JST XH, J3 JST XH, J4 JST XH, K1 G6A-274P, K2 G6A-274P, Q1 BC847/547, Q2 BC847/547, U1 SFH6206-2

Commit message: Updated to 3.30; See README.md
Parts:
- D1, D2: footprint (none) -> Diode_SMD:D_SOD-123
